File: kicad/neurx.kicad_sch (KiCad schematic)
At the start: 154 parts, among them P0 Keyswitch, P1 Keyswitch, U1 Raspberry_Pi_Pico

Commit message: Add files via upload
Parts:
- added D68, D77, D79, D80, D81, D82, D83, D84: Diode, ScottoKeebs_Components:Diode_DO-35, symbol ScottoKeebs:Placeholder_Diode
- added I2, I4, T1, T2, T3, T4, T5: Keyswitch, ScottoKeebs_MX:MX_PCB_1.00u, symbol ScottoKeebs:Placeholder_Keyswitch
- added S42: Keyswitch, ScottoKeebs_MX:MX_PCB_1.25u, symbol ScottoKeebs:Placeholder_Keyswitch
- I1: renamed from S75; footprint ScottoKeebs_MX:MX_PCB_1.25u -> ScottoKeebs_MX:MX_PCB_1.00u
- I3: renamed from S76; footprint ScottoKeebs_MX:MX_PCB_1.25u -> ScottoKeebs_MX:MX_PCB_1.00u
- S22: renamed from S72; footprint ScottoKeebs_MX:MX_PCB_6.25u -> ScottoKeebs_MX:MX_PCB_5.50u
- S45: renamed from S69; footprint ScottoKeebs_MX:MX_PCB_2.75u -> ScottoKeebs_MX:MX_PCB_1.75u
- renumbered S29 to B1, D3 to D10, D18 to D11, D31 to D12, D45 to D13, D58 to D14, D4 to D15, D19 to D16, D32 to D17, D46 to D18, D59 to D19, D16 to D2, D71 to D20, D5 to D21, D20 to D22, D33 to D23, D47 to D24, D60 to D25, D6 to D26, D21 to D27, D34 to D28, D48 to D29, D30 to D3, D61 to D30, D7 to D31, D22 to D32, D35 to D33, D49 to D34, D62 to D35, D72 to D36, D8 to D37, D23 to D38, D36 to D39, D44 to D4, D50 to D40, D63 to D41, D9 to D42, D24 to D43, D37 to D44, D51 to D45, D64 to D46, D10 to D47, D25 to D48, D38 to D49, D68 to D5, D52 to D50, D65 to D51, D73 to D52, D11 to D53, D26 to D54, D39 to D55, D53 to D56, D66 to D57, D12 to D58, D27 to D59, D2 to D6, D40 to D60, D54 to D61, D67 to D62, D74 to D63, D13 to D64, D28 to D65, D41 to D66, D55 to D67, D14 to D69, D17 to D7, D42 to D70, D57 to D71, D69 to D72, D75 to D73, D15 to D74, D29 to D75, D43 to D76, D76 to D78, D56 to D8, D70 to D9, Esc1 to E1, S16 to K1, S25 to K10, S26 to K11, S27 to K12, S28 to K13, S17 to K2, S18 to K3, S19 to K4, S20 to K5, S21 to K6, S22 to K7, S23 to K8, S24 to K9, P0 to P1, P1 to P2, S30 to S1, S46 to S10, S59 to S11, S71 to S12, S33 to S13, S47 to S14, S60 to S15, S34 to S16, S48 to S17, S61 to S18, S35 to S19, S44 to S2, S49 to S20, S62 to S21, S36 to S23, S50 to S24, S63 to S25, S37 to S26, S51 to S27, S64 to S28, S38 to S29, S68 to S3, S52 to S30, S65 to S31, S73 to S32, S39 to S33, S53 to S34, S66 to S35, S40 to S36, S54 to S37, S67 to S38, S74 to S39, S56 to S4, S41 to S40, S55 to S41, S42 to S43, S57 to S44, S43 to S46, S70 to S5, S31 to S6, S45 to S7, S58 to S8, S32 to S9
Connections:
- net Col 0: no longer U1.1 (GPIO0)
- net Col 1: no longer U1.2 (GPIO1)
- net Col 10: no longer S32.1, U1.14 (GPIO10)
- net Col 11: no longer U1.15 (GPIO11)
- net Col 12: now also S42.1; no longer U1.16 (GPIO12)
- net Col 13: no longer U1.17 (GPIO13)
- net Col 14: now also I2.1; no longer U1.19 (GPIO14)
- net Col 2: no longer U1.4 (GPIO2)
- net Col 3: no longer U1.5 (GPIO3)
- net Col 4: no longer U1.6 (GPIO4)
- net Col 5: no longer U1.7 (GPIO5)
- net Col 6: no longer U1.9 (GPIO6)
- net Col 7: no longer U1.10 (GPIO7)
- net Col 8: no longer U1.11 (GPIO8)
- net Col 9: now also S32.1; no longer U1.12 (GPIO9)
- net Row 0: now also D79.1 (K)
- net Row 1: now also D80.1 (K)
- net Row 2: now also D81.1 (K)
- net Row 3: now also D82.1 (K)
- net Row 4: now also D77.1 (K), D83.1 (K)
- net Row 5: now also D68.1 (K), D84.1 (K)
- new net: D81.2 (A), T3.2
- new net: D68.2 (A), S42.2
- new net: D82.2 (A), T4.2
- new net: D80.2 (A), T2.2
- new net: D83.2 (A), T5.2
- new net: D77.2 (A), I2.2
- new net: D79.2 (A), T1.2
- new net: D84.2 (A), I4.2
- new net Col 15: I4.1, T1.1, T2.1, T3.1, T4.1, T5.1
Other:
- moved on the sheet: B1, D1, D10, D11, D12, D13, D14, D15, D16, D17, D18, D19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

Commit message: Add files via upload
Parts:
- removed D68: Diode, ScottoKeebs_Components:Diode_DO-35, symbol ScottoKeebs:Placeholder_Diode
- removed S42: Keyswitch, ScottoKeebs_MX:MX_PCB_1.25u, symbol ScottoKeebs:Placeholder_Keyswitch
- S22: footprint ScottoKeebs_MX:MX_PCB_5.50u -> ScottoKeebs_MX:MX_PCB_6.25u
- renumbered D69 to D68, D70 to D69, D71 to D70, D72 to D71, D73 to D72, D74 to D73, D75 to D74, D76 to D75, D77 to D76, D78 to D77, D79 to D78, D80 to D79, D81 to D80, D82 to D81, D83 to D82, D84 to D83, S43 to S42, S44 to S43, S45 to S44, S46 to S45
Connections:
- net Col 0: now also U1.20 (GPIO15)
- net Col 1: now also U1.19 (GPIO14)
- net Col 10: now also U1.7 (GPIO5)
- net Col 11: now also U1.6 (GPIO4)
- net Col 12: now also U1.5 (GPIO3)
- net Col 13: now also U1.4 (GPIO2)
- net Col 14: now also U1.2 (GPIO1)
- net Col 15: now also U1.1 (GPIO0)
- net Col 2: now also U1.17 (GPIO13)
- net Col 3: now also U1.16 (GPIO12)
- net Col 4: now also U1.15 (GPIO11)
- net Col 5: now also U1.14 (GPIO10)
- net Col 6: now also U1.12 (GPIO9)
- net Col 7: now also U1.11 (GPIO8)
- net Col 8: now also U1.10 (GPIO7)
- net Col 9: now also U1.9 (GPIO6)

Commit message: Plug row 5 to pico, completely forgot that
Connections:
- net Row 5: now also U1.27 (GPIO21)
Changed lines of the file:
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@@
+		)
+	)
+	(global_label "Row 5"
+		(shape input)
+		(at 368.3 109.22 180)
+		(fields_autoplaced yes)
+		(effects
+			(font
+				(size 1.27 1.27)
+			)
+			(justify right)
+		)
+		(property "Intersheetrefs" "${INTERSHEET_REFS}"
+			(at 359.3882 109.22 0)
+			(effects
+				(font
+					(size 1.27 1.27)
+				)
+				(justify right)
+				(hide yes)
+			)
 		)
 	)
