File: kicad/neurx.kicad_pcb (KiCad board)
At the start: 2 copper layers, 297.2 x 152.4 mm, 159 parts, among them P0 Keyswitch, P1 Keyswitch, U1 Raspberry_Pi_Pico

Commit message: Add files via upload
Parts:
- removed the REF** at (196.9, 203.3)
- removed the REF** at (325.5, 184.3)
- added D68: Diode, ScottoKeebs_Components:Diode_DO-35, B.Cu at (313.6, 205.9)
- added D77: Diode, ScottoKeebs_Components:Diode_DO-35, B.Cu at (351.7, 186.8)
- added D79: Diode, ScottoKeebs_Components:Diode_DO-35, B.Cu at (370.7, 110.6)
- added D80: Diode, ScottoKeebs_Components:Diode_DO-35, B.Cu at (370.7, 129.7)
- added D81: Diode, ScottoKeebs_Components:Diode_DO-35, B.Cu at (370.7, 148.7)
- added D82: Diode, ScottoKeebs_Components:Diode_DO-35, B.Cu at (370.7, 167.8)
- added D83: Diode, ScottoKeebs_Components:Diode_DO-35, B.Cu at (370.7, 186.8)
- added D84: Diode, ScottoKeebs_Components:Diode_DO-35, B.Cu at (370.7, 205.9)
- added I2: Keyswitch, ScottoKeebs_MX:MX_PCB_1.00u, F.Cu at (342.1, 184.3)
- added I4: Keyswitch, ScottoKeebs_MX:MX_PCB_1.00u, F.Cu at (361.2, 203.3)
- added S42: Keyswitch, ScottoKeebs_MX:MX_PCB_1.25u, F.Cu at (301.7, 203.3)
- added T1: Keyswitch, ScottoKeebs_MX:MX_PCB_1.00u, F.Cu at (361.2, 108.1)
- added T2: Keyswitch, ScottoKeebs_MX:MX_PCB_1.00u, F.Cu at (361.2, 127.1)
- added T3: Keyswitch, ScottoKeebs_MX:MX_PCB_1.00u, F.Cu at (361.2, 146.2)
- added T4: Keyswitch, ScottoKeebs_MX:MX_PCB_1.00u, F.Cu at (361.2, 165.2)
- added T5: Keyswitch, ScottoKeebs_MX:MX_PCB_1.00u, F.Cu at (361.2, 184.3)
- I1: renamed from S75; footprint ScottoKeebs_MX:MX_PCB_1.25u -> ScottoKeebs_MX:MX_PCB_1.00u
- I3: renamed from S76; footprint ScottoKeebs_MX:MX_PCB_1.25u -> ScottoKeebs_MX:MX_PCB_1.00u
- S22: renamed from S72; footprint ScottoKeebs_MX:MX_PCB_6.25u -> ScottoKeebs_MX:MX_PCB_5.50u
- S45: renamed from S69; footprint ScottoKeebs_MX:MX_PCB_2.75u -> ScottoKeebs_MX:MX_PCB_1.75u
- moved U1 31.1 mm to (294.5, 83.3)
- moved D72 19.1 mm to (332.6, 186.8)
- moved D52 14.3 mm to (265.9, 205.9)
- moved D36 14.3 mm to (242.1, 205.9)
- moved S32 14.3 mm to (254.0, 203.3)
- moved S39 14.3 mm to (277.8, 203.3)
- moved D63 14.3 mm to (289.7, 205.9)
- moved S45 9.53 mm to (315.9, 184.3)
- moved I1 7.14 mm to (323.1, 203.3)
- moved S22 7.14 mm to (189.7, 203.3)
- moved D73 4.76 mm to (332.6, 205.9)
- moved I3 2.38 mm to (342.1, 203.3)
- renumbered S29 to B1, D3 to D10, D18 to D11, D31 to D12, D45 to D13, D58 to D14, D4 to D15, D19 to D16, D32 to D17, D46 to D18, D59 to D19, D16 to D2, D71 to D20, D5 to D21, D20 to D22, D33 to D23, D47 to D24, D60 to D25, D6 to D26, D21 to D27, D34 to D28, D48 to D29, D30 to D3, D61 to D30, D7 to D31, D22 to D32, D35 to D33, D49 to D34, D62 to D35, D72 to D36, D8 to D37, D23 to D38, D36 to D39, D44 to D4, D50 to D40, D63 to D41, D9 to D42, D24 to D43, D37 to D44, D51 to D45, D64 to D46, D10 to D47, D25 to D48, D38 to D49, D68 to D5, D52 to D50, D65 to D51, D73 to D52, D11 to D53, D26 to D54, D39 to D55, D53 to D56, D66 to D57, D12 to D58, D27 to D59, D2 to D6, D40 to D60, D54 to D61, D67 to D62, D74 to D63, D13 to D64, D28 to D65, D41 to D66, D55 to D67, D14 to D69, D17 to D7, D42 to D70, D57 to D71, D69 to D72, D75 to D73, D15 to D74, D29 to D75, D43 to D76, D76 to D78, D56 to D8, D70 to D9, Esc1 to E1, S16 to K1, S25 to K10, S26 to K11, S27 to K12, S28 to K13, S17 to K2, S18 to K3, S19 to K4, S20 to K5, S21 to K6, S22 to K7, S23 to K8, S24 to K9, P0 to P1, P1 to P2, S30 to S1, S46 to S10, S59 to S11, S71 to S12, S33 to S13, S47 to S14, S60 to S15, S34 to S16, S48 to S17, S61 to S18, S35 to S19, S44 to S2, S49 to S20, S62 to S21, S36 to S23, S50 to S24, S63 to S25, S37 to S26, S51 to S27, S64 to S28, S38 to S29, S68 to S3, S52 to S30, S65 to S31, S73 to S32, S39 to S33, S53 to S34, S66 to S35, S40 to S36, S54 to S37, S67 to S38, S74 to S39, S56 to S4, S41 to S40, S55 to S41, S42 to S43, S57 to S44, S43 to S46, S70 to S5, S31 to S6, S45 to S7, S58 to S8, S32 to S9
Connections:
- S32 pad 1: Col 10 -> Col 9
- U1 pad 1: Col 0 -> unconnected-(U1-GPIO0-Pad1)
- U1 pad 10: Col 7 -> unconnected-(U1-GPIO7-Pad10)
- U1 pad 11: Col 8 -> unconnected-(U1-GPIO8-Pad11)
- U1 pad 12: Col 9 -> unconnected-(U1-GPIO9-Pad12)
- U1 pad 14: Col 10 -> unconnected-(U1-GPIO10-Pad14)
- U1 pad 15: Col 11 -> unconnected-(U1-GPIO11-Pad15)
- U1 pad 16: Col 12 -> unconnected-(U1-GPIO12-Pad16)
- U1 pad 17: Col 13 -> unconnected-(U1-GPIO13-Pad17)
- U1 pad 19: Col 14 -> unconnected-(U1-GPIO14-Pad19)
- U1 pad 2: Col 1 -> unconnected-(U1-GPIO1-Pad2)
- U1 pad 4: Col 2 -> unconnected-(U1-GPIO2-Pad4)
- U1 pad 5: Col 3 -> unconnected-(U1-GPIO3-Pad5)
- U1 pad 6: Col 4 -> unconnected-(U1-GPIO4-Pad6)
- U1 pad 7: Col 5 -> unconnected-(U1-GPIO5-Pad7)
- U1 pad 9: Col 6 -> unconnected-(U1-GPIO6-Pad9)
Routing:
- net Col 15: track 0.00 -> 146.9 mm
- net Col 0: track 396.8 -> 311.8 mm
- net Col 1: track 378.8 -> 299.3 mm
- net Col 2: track 336.3 -> 267.8 mm
- net Col 3: track 338.3 -> 274.7 mm
- net Col 4: track 292.5 -> 234.2 mm
- net Row 3: track 417.6 -> 363.0 mm, vias 0 -> 1
- net Col 5: track 270.5 -> 217.7 mm
- net Col 6: track 266.1 -> 225.6 mm
- net Col 7: track 224.1 -> 187.2 mm
- net Row 4: track 399.5 -> 365.8 mm, vias 0 -> 1
- net Col 10: track 175.9 -> 144.3 mm
- net Col 8: track 202.2 -> 170.7 mm
- net Col 12: track 110.0 -> 140.6 mm
- net Row 2: track 321.1 -> 346.6 mm
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Other:
- board size 297.2 x 152.4 mm -> 316.2 x 152.4 mm

Commit message: Add files via upload
Parts:
- removed the D68 at (313.6, 205.9)
- removed the S42 at (301.7, 203.3)
- S22: footprint ScottoKeebs_MX:MX_PCB_5.50u -> ScottoKeebs_MX:MX_PCB_6.25u
- moved D52 14.3 mm to (280.2, 205.9)
- moved D36 14.3 mm to (256.4, 205.9)
- moved S32 14.3 mm to (268.3, 203.3)
- moved S39 14.3 mm to (292.1, 203.3)
- moved D63 14.3 mm to (304.0, 205.9)
- moved S22 7.14 mm to (196.9, 203.3)
- renumbered D69 to D68, D70 to D69, D71 to D70, D72 to D71, D73 to D72, D74 to D73, D75 to D74, D76 to D75, D77 to D76, D78 to D77, D79 to D78, D80 to D79, D81 to D80, D82 to D81, D83 to D82, D84 to D83, S43 to S42, S44 to S43, S45 to S44, S46 to S45
Connections:
- U1 pad 1: unconnected-(U1-GPIO0-Pad1) -> Col 15
- U1 pad 10: unconnected-(U1-GPIO7-Pad10) -> Col 8
- U1 pad 11: unconnected-(U1-GPIO8-Pad11) -> Col 7
- U1 pad 12: unconnected-(U1-GPIO9-Pad12) -> Col 6
- U1 pad 14: unconnected-(U1-GPIO10-Pad14) -> Col 5
- U1 pad 15: unconnected-(U1-GPIO11-Pad15) -> Col 4
- U1 pad 16: unconnected-(U1-GPIO12-Pad16) -> Col 3
- U1 pad 17: unconnected-(U1-GPIO13-Pad17) -> Col 2
- U1 pad 19: unconnected-(U1-GPIO14-Pad19) -> Col 1
- U1 pad 2: unconnected-(U1-GPIO1-Pad2) -> Col 14
- U1 pad 20: unconnected-(U1-GPIO15-Pad20) -> Col 0
- U1 pad 4: unconnected-(U1-GPIO2-Pad4) -> Col 13
- U1 pad 5: unconnected-(U1-GPIO3-Pad5) -> Col 12
- U1 pad 6: unconnected-(U1-GPIO4-Pad6) -> Col 11
- U1 pad 7: unconnected-(U1-GPIO5-Pad7) -> Col 10
- U1 pad 9: unconnected-(U1-GPIO6-Pad9) -> Col 9
Routing:
- net Col 12: track 140.6 -> 99.5 mm
- net Net-(D63-A): track 19.6 -> 9.36 mm
- net Net-(D68-A) (its old number): track 9.37 -> 0.00 mm
- net Net-(D36-A): track 49.8 -> 57.0 mm
- net Col 9: track 174.2 -> 180.2 mm
- net Col 11: track 151.4 -> 147.5 mm
- net Col 6: track 225.6 -> 224.7 mm

Commit message: Update design from sketch
Connections:
- U1 pad 27: unconnected-(U1-GPIO21-Pad27) -> Row 5
Routing:
- net Row 5: track 281.0 -> 405.0 mm, vias 0 -> 1
